File: Genli.kicad_sch (KiCad schematic)
At the start: 10 parts, among them U1 ICM-20948, U2 VL53L0X, U3 VL53L0X, U9 BUCK_5V

Commit message: revamp esp symbols and finalize schematic (erc passed)
Parts:
- removed U4, U5, U6, U7: (no value), symbol Genli:ESC_30A
- added U11, U13, U5, U6: (no value), symbol Genli:ESC_30A_SIGNAL
- added U12, U14, U4, U7: (no value), symbol Genli:ESC_30A_Power
Connections:
- net ESC1_SIG: now also U5.1 (SIGNAL)
- net ESC2_SIG: now also U6.1 (SIGNAL)
- net ESC3_SIG: now also U13.1 (SIGNAL)
- net ESC4_SIG: now also U11.1 (SIGNAL)
- net GND: now also U11.2 (GND), U12.2 (BAT-), U13.2 (GND), U14.2 (BAT-), U4.2 (BAT-), U5.2 (GND), U6.2 (GND), U7.2 (BAT-)
- net VBAT: now also U12.1 (BAT+), U14.1 (BAT+), U4.1 (BAT+), U7.1 (BAT+)

Commit message: assign all footprints
Parts:
- removed U9: BUCK_5V, symbol Genli:uctronic_buck_converter
- added U15: (no value), PCM_SparkFun-Connector:ScrewTerminal_1x02_P5.0mm, symbol Genli:buck_output
- added U9: (no value), PCM_SparkFun-Connector:ScrewTerminal_1x02_P5.0mm, symbol Genli:buck_input
- U1: footprint (none) -> HopCopter:SEN-15335
- U10: footprint ESP32_30pin -> PCM_SparkFun-RF:ESP32-WROOM-32D-DFM_PASTE
- U11, U13, U5, U6: footprint (none) -> Connector_PinHeader_2.54mm:PinHeader_1x02_P2.54mm_Vertical
- U12, U14, U4, U7: footprint (none) -> PCM_SparkFun-Connector:ScrewTerminal_1x02_P5.0mm
- U2, U3: footprint (none) -> Connector_PinHeader_2.54mm:PinHeader_1x06_P2.54mm_Vertical
- U8: footprint (none) -> Connector_AMASS:AMASS_XT60-F_1x02_P7.20mm_Vertical
Connections:
- net GND: now also U9.2 (VIN-)
- net VBAT: now also U9.1 (VIN+)
- net at U10.1 (VIN): now also U15.1 (5V)
- net at U10.17 (GND): now also U15.2 (GND)

Commit message: update schematic with on-off switch adapter and update pcb design with matching footprints
Parts:
- added J1: Screw_Terminal_01x02, PCM_SparkFun-Connector:ScrewTerminal_1x02_P5.0mm, symbol Connector:Screw_Terminal_01x02
- U10: footprint PCM_SparkFun-RF:ESP32-WROOM-32D-DFM_PASTE -> ESP32_Footprints:ESP32_30pin
- U8: footprint Connector_AMASS:AMASS_XT60-F_1x02_P7.20mm_Vertical -> Connector_AMASS:AMASS_XT60PW-F_1x02_P7.20mm_Horizontal
Connections:
- net GND: now also U8.2 (BAT-); no longer U8.BAT- (2)
- net VBAT: now also J1.2 (Pin_2); no longer U8.BAT+ (1)
- new net: J1.1 (Pin_1), U8.1 (BAT+)
Other:
- note added: "switch goes here"
Changed lines of the file:
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@@
 	(text "Battery\n"
 		(exclude_from_sim no)
-		(at 185.166 18.542 0)
+		(at 201.168 20.828 0)
 		(effects
 			(font
@@
 		)
 	)
+	(text "switch goes here"
+		(exclude_from_sim no)
+		(at 186.69 51.054 0)
+		(effects
+			(font
+				(size 1.27 1.27)
+			)
+		)
+	)
 	(no_connect
 		(at 72.39 90.17)
@@
 	(wire
 		(pts
+			(xy 165.1 34.29) (xy 176.53 34.29)
+		)
+		(stroke
+			(width 0)
+			(type default)
+		)
+	)
+	(wire
+		(pts
 			(xy 220.98 77.47) (xy 220.98 81.28)
 		)
@@
 	(wire
 		(pts
+			(xy 185.42 40.64) (xy 176.53 40.64)
+		)
+		(stroke
+			(width 0)
+			(type default)
+		)
+	)
+	(wire
+		(pts
 			(xy 220.98 106.68) (xy 237.49 106.68)
 		)
@@
 	(wire
 		(pts
-			(xy 170.18 26.67) (xy 176.53 26.67)
+			(xy 170.18 26.67) (xy 233.68 26.67)
 		)
 		(stroke
@@
 	(wire
 		(pts
+			(xy 187.96 40.64) (xy 201.93 40.64)
+		)
+		(stroke
+			(width 0)
+			(type default)
+		)
+	)
+	(wire
+		(pts
 			(xy 99.06 78.74) (xy 102.87 78.74)
 		)
@@
 	(wire
 		(pts
+			(xy 201.93 34.29) (xy 233.68 34.29)
+		)
+		(stroke
+			(width 0)
+			(type default)
+		)
+	)
+	(wire
+		(pts
 			(xy 132.08 66.04) (xy 137.16 66.04)
 		)
@@
 	(wire
 		(pts
-			(xy 170.18 34.29) (xy 176.53 34.29)
+			(xy 201.93 40.64) (xy 201.93 34.29)
 		)
 		(stroke
@@
 		(pts
 			(xy 106.68 100.33) (xy 110.49 100.33)
+		)
+		(stroke
+			(width 0)
+			(type default)
+		)
+	)
+	(wire
+		(pts
+			(xy 176.53 40.64) (xy 176.53 34.29)
 		)
 		(stroke
@@
 	)
 	(label "VBAT"
-		(at 170.18 34.29 180)
+		(at 165.1 34.29 180)
 		(effects
 			(font
@@
 	)
 	(symbol
+		(lib_id "Genli:battery_conn")
+		(at 242.57 30.48 90)
+		(unit 1)
+		(body_style 1)
+		(exclude_from_sim no)
+		(in_bom yes)
+		(on_board yes)
+		(in_pos_files yes)
+		(dnp no)
+		(fields_autoplaced yes)
+		(property "Reference" "U8"
+			(at 252.73 30.4799 90)
+			(show_name no)
+			(do_not_autoplace no)
+			(effects
+				(font
+					(size 1.27 1.27)
+				)
+				(justify right)
+			)
+		)
+		(property "Value" ""
+			(at 242.57 30.48 0)
+			(show_name no)
+			(do_not_autoplace no)
+			(effects
+				(font
+					(size 1.27 1.27)
+				)
+			)
+		)
+		(property "Footprint" "Connector_AMASS:AMASS_XT60PW-F_1x02_P7.20mm_Horizontal"
+			(at 242.57 30.48 0)
+			(hide yes)
+			(show_name no)
+			(do_not_autoplace no)
+			(effects
+				(font
+					(size 1.27 1.27)
+				)
+			)
+		)
+		(property "Datasheet" ""
+			(at 242.57 30.48 0)
+			(hide yes)
+			(show_name no)
+			(do_not_autoplace no)
+			(effects
+				(font
+					(size 1.27 1.27)
+				)
+			)
+		)
+		(property "Description" ""
+			(at 242.57 30.48 0)
+			(hide yes)
+			(show_name no)
+			(do_not_autoplace no)
+			(effects
+				(font
+					(size 1.27 1.27)
+				)
+			)
+		)
+		(pin "1"
+		)
+		(pin "2"
+		)
+		(instances
+			(project "Genli"
+				(path "/ab1ba344-0bbc-4d03-a791-b040cd8e0018"
+					(reference "U8")
+					(unit 1)
+				)
+			)
+		)
+	)
+	(symbol
 		(lib_id "Genli:ESC_30A_SIGNAL")
 		(at 177.8 88.9 0)
@@
 			)
 		)
-		(property "Footprint" "PCM_SparkFun-RF:ESP32-WROOM-32D-DFM_PASTE"
+		(property "Footprint" "ESP32_Footprints:ESP32_30pin"
 			(at 55.88 80.01 0)
 			(show_name no)
@@
 	)
 	(symbol
+		(lib_id "Connector:Screw_Terminal_01x02")
+		(at 187.96 45.72 270)
+		(unit 1)
+		(body_style 1)
+		(exclude_from_sim no)
+		(in_bom yes)
+		(on_board yes)
+		(in_pos_files yes)
+		(dnp no)
+		(fields_autoplaced yes)
+		(property "Reference" "J1"
+			(at 190.5 44.4499 90)
+			(show_name no)
+			(do_not_autoplace no)
+			(effects
+				(font
+					(size 1.27 1.27)
+				)
+				(justify left)
+			)
+		)
+		(property "Value" "Screw_Terminal_01x02"
+			(at 190.5 46.9899 90)
+			(show_name no)
+			(do_not_autoplace no)
+			(effects
+				(font
+					(size 1.27 1.27)
+				)
+				(justify left)
+			)
+		)
+		(property "Footprint" "PCM_SparkFun-Connector:ScrewTerminal_1x02_P5.0mm"
+			(at 187.96 45.72 0)
+			(hide yes)
+			(show_name no)
+			(do_not_autoplace no)
+			(effects
+				(font
+					(size 1.27 1.27)
+				)
+			)
+		)
+		(property "Datasheet" ""
+			(at 187.96 45.72 0)
+			(hide yes)
+			(show_name no)
+			(do_not_autoplace no)
+			(effects
+				(font
+					(size 1.27 1.27)
+				)
+			)
+		)
+		(property "Description" "Generic screw terminal, single row, 01x02, script generated (kicad-library-utils/schlib/autogen/connector/)"
+			(at 187.96 45.72 0)
+			(hide yes)
+			(show_name no)
+			(do_not_autoplace no)
+			(effects
+				(font
+					(size 1.27 1.27)
+				)
+			)
+		)
+		(pin "2"
+		)
+		(pin "1"
+		)
+		(instances
+			(project "Genli"
+				(path "/ab1ba344-0bbc-4d03-a791-b040cd8e0018"
+					(reference "J1")
+					(unit 1)
+				)
+			)
+		)
+	)
+	(symbol
 		(lib_id "Genli:buck_input")
 		(at 105.41 35.56 0)
@@
 					(unit 1)
 				)
-			)
-		)
-	)
-	(symbol
-		(lib_id "Genli:battery_conn")
-		(at 185.42 30.48 90)
-		(unit 1)
-		(body_style 1)
-		(exclude_from_sim no)
-		(in_bom yes)
-		(on_board yes)
-		(in_pos_files yes)
-		(dnp no)
-		(fields_autoplaced yes)
-		(property "Reference" "U8"
-			(at 195.58 30.4799 90)
-			(show_name no)
-			(do_not_autoplace no)
-			(effects
-				(font
-					(size 1.27 1.27)
-				)
-				(justify right)
-			)
-		)
-		(property "Value" ""
-			(at 185.42 30.48 0)
-			(show_name no)
-			(do_not_autoplace no)
-			(effects
-				(font
-					(size 1.27 1.27)
-				)
-			)
-		)
-		(property "Footprint" "Connector_AMASS:AMASS_XT60-F_1x02_P7.20mm_Vertical"
-			(at 185.42 30.48 0)
-			(hide yes)
-			(show_name no)
-			(do_not_autoplace no)
-			(effects
-				(font
-					(size 1.27 1.27)
-				)
-			)
-		)
-		(property "Datasheet" ""
-			(at 185.42 30.48 0)
-			(hide yes)
-			(show_name no)
-			(do_not_autoplace no)
-			(effects
-				(font
-					(size 1.27 1.27)
-				)
-			)
-		)
-		(property "Description" ""
-			(at 185.42 30.48 0)
-			(hide yes)
-			(show_name no)
-			(do_not_autoplace no)
-			(effects
-				(font
-					(size 1.27 1.27)
-				)
-			)
-		)
-		(pin "BAT+"
-		)
-		(pin "BAT-"
-		)
-		(instances
-			(project "Genli"
-				(path "/ab1ba344-0bbc-4d03-a791-b040cd8e0018"
-					(reference "U8")
-					(unit 1)
-				)

Commit message: update pcb layout with cleaner traces; switch esc +/- connectors to soldered pad instead of screw terminal
Parts:
- U12, U14, U4, U7: footprint PCM_SparkFun-Connector:ScrewTerminal_1x02_P5.0mm -> HopCopter:ESC_Power_SolderPads_1x02
Changed lines of the file:
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@@
+	)
+	(no_connect
+		(at 125.73 105.41)
+	)
+	(no_connect
+		(at 44.45 87.63)
+	)
+	(no_connect
+		(at 72.39 67.31)
+	)
+	(no_connect
+		(at 44.45 67.31)
+	)
+	(no_connect
+		(at 72.39 77.47)
+	)
+	(no_connect
+		(at 44.45 95.25)
+	)
+	(no_connect
+		(at 125.73 92.71)
+	)
+	(no_connect
+		(at 125.73 95.25)
+	)
+	(no_connect
+		(at 72.39 92.71)
+	)
+	(no_connect
+		(at 72.39 74.93)
+	)
+	(no_connect
+		(at 72.39 69.85)
+	)
+	(no_connect
+		(at 44.45 97.79)
 	)
 	(no_connect
@@
 	)
 	(no_connect
-		(at 125.73 105.41)
-	)
-	(no_connect
-		(at 44.45 87.63)
-	)
-	(no_connect
-		(at 72.39 67.31)
-	)
-	(no_connect
-		(at 44.45 67.31)
-	)
-	(no_connect
-		(at 72.39 77.47)
-	)
-	(no_connect
-		(at 44.45 95.25)
-	)
-	(no_connect
-		(at 125.73 92.71)
-	)
-	(no_connect
-		(at 125.73 95.25)
-	)
-	(no_connect
-		(at 72.39 92.71)
-	)
-	(no_connect
-		(at 72.39 74.93)
-	)
-	(no_connect
-		(at 72.39 69.85)
-	)
-	(no_connect
-		(at 44.45 97.79)
-	)
-	(no_connect
 		(at 137.16 76.2)
 	)
@@
 	(wire
 		(pts
-			(xy 83.82 64.77) (xy 72.39 64.77)
-		)
-		(stroke
-			(width 0)
-			(type default)
-		)
-	)
-	(wire
-		(pts
 			(xy 171.45 71.12) (xy 187.96 71.12)
 		)
@@
 	(wire
 		(pts
-			(xy 83.82 50.8) (xy 127 50.8)
-		)
-		(stroke
-			(width 0)
-			(type default)
-		)
-	)
-	(wire
-		(pts
 			(xy 44.45 48.26) (xy 44.45 62.23)
 		)
@@
 	(wire
 		(pts
+			(xy 72.39 50.8) (xy 72.39 64.77)
+		)
+		(stroke
+			(width 0)
+			(type default)
+		)
+	)
+	(wire
+		(pts
 			(xy 222.25 72.39) (xy 238.76 72.39)
 		)
@@
 	(wire
 		(pts
-			(xy 83.82 50.8) (xy 83.82 64.77)
-		)
-		(stroke
-			(width 0)
-			(type default)
-		)
-	)
-	(wire
-		(pts
 			(xy 106.68 97.79) (xy 110.49 97.79)
 		)
@@
 	(wire
 		(pts
+			(xy 127 38.1) (xy 127 50.8)
+		)
+		(stroke
+			(width 0)
+			(type default)
+		)
+	)
+	(wire
+		(pts
 			(xy 44.45 48.26) (xy 129.54 48.26)
 		)
@@
 	(wire
 		(pts
-			(xy 127 50.8) (xy 127 38.1)
+			(xy 127 50.8) (xy 72.39 50.8)
 		)
 		(stroke
@@
 			)
 		)
-		(property "Footprint" "PCM_SparkFun-Connector:ScrewTerminal_1x02_P5.0mm"
+		(property "Footprint" "HopCopter:ESC_Power_SolderPads_1x02"
 			(at 246.38 109.22 0)
 			(hide yes)
@@
 			)
 		)
-		(property "Footprint" "PCM_SparkFun-Connector:ScrewTerminal_1x02_P5.0mm"
+		(property "Footprint" "HopCopter:ESC_Power_SolderPads_1x02"
 			(at 247.65 74.93 0)
 			(hide yes)
@@
 			)
 		)
-		(property "Footprint" "PCM_SparkFun-Connector:ScrewTerminal_1x02_P5.0mm"
+		(property "Footprint" "HopCopter:ESC_Power_SolderPads_1x02"
 			(at 196.85 110.49 0)
 			(hide yes)
@@
 			)
 		)
-		(property "Footprint" "PCM_SparkFun-Connector:ScrewTerminal_1x02_P5.0mm"
+		(property "Footprint" "HopCopter:ESC_Power_SolderPads_1x02"
 			(at 196.85 78.74 0)
 			(hide yes)
