File: v1-prototype/Genli.kicad_sch (KiCad schematic)
At the start: 16 parts, among them J1 Screw_Terminal_01x02, U1 ICM-20948, U2 VL53L0X, U3 VL53L0X

Commit message: Correct the regulator to five pins and move the power switch to SHDN
The Pololu D24V10F5 has five connections -- VIN, GND, VOUT, SHDN and PG -- not
the three this spec assumed. That changes its symbol and footprint, and it
changes the power switch.

SHDN pulled low shuts the regulator down, so J8 moves from the BAT path onto
SHDN. Switching SHDN is signal level: no current, no raw pack voltage on a
mechanical contact a crash can knock, and nothing in series with the supply to
add resistance or fail open. The trade is that BAT stays present when switched
off and the divider keeps drawing ~138 uA, which is irrelevant beside pack
self-discharge. Leaving J8 unfitted is now the do-nothing default rather than
something that has to be jumpered closed.

Adds the electrical types for the custom symbol -- VOUT as a power output in
particular, since that is what stops ERC reporting the +5V net as undriven --
and a note that BAT and GND need PWR_FLAGs because they arrive through a
connector's passive pins. Records that the physical pin order must come from
Pololu's dimension diagram; it is printed on the back of the module and is not
reliably documented anywhere in text.

Also rewrites the cross-repository doc links as URLs. They were relative paths
from when this spec lived in the Revali tree and have been broken since the
split.

Co-Authored-By: Claude Opus 5 <noreply@anthropic.com>
Connections:
- no-connect marks 21 -> 23
Changed lines of the file:
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@@
+	)
+	(no_connect
+		(at 238.76 29.21)
 	)
 	(no_connect
@@
 	)
 	(no_connect
+		(at 240.03 43.18)
+	)
+	(no_connect
